Commit message: Create lawn world

File: jackal_ws/src/jackal/jackal_description/urdf/jackal.urdf.xacro (robot description, xacro)
@@ -63,5 +63,5 @@
     <transmission name="${prefix}_wheel_trans">
       <type>transmission_interface/SimpleTransmission</type>
-      <joint name="${prefix}_wheel">
+      <joint name="${prefix}_wheel_joint">
         <hardwareInterface>hardware_interface/VelocityJointInterface</hardwareInterface>
       </joint>

Commit message: fixed imu sensor and created ultrasonic sensor to detect grass height

File: jackal_ws/src/jackal/jackal_description/urdf/jackal.urdf.xacro (robot description, xacro)
@@ -256,4 +256,56 @@
     </joint>
   </ros2_control>
+  <!-- Ultrasonic -->
+  <link name="ultrasonic_link">
+    <visual>
+        <origin xyz="0 0 0" rpy="0 0 0"/>
+        <geometry>
+        <cylinder radius="0.015" length="0.02"/>
+        </geometry>
+        <material name="black"/>
+    </visual>
+    <inertial>
+        <mass value="0.01"/>
+        <origin xyz="0 0 0" rpy="0 0 0"/>
+        <inertia ixx="1e-6" ixy="0.0" ixz="0.0" iyy="1e-6" iyz="0.0" izz="1e-6"/>
+    </inertial>
+  </link>
+  <joint name="ultrasonic_joint" type="fixed">
+    <parent link="chassis_link"/>
+    <child link="ultrasonic_link"/>
+    <origin xyz="0 0 -0.02" rpy="0 1.5708 0"/>
+  </joint>
+  <gazebo reference="ultrasonic_link">
+    <selfCollide>false</selfCollide>
+    <sensor type="ray" name="ultrasonic_sensor">
+        <pose>0 0 0 0 0 0</pose>
+        <visualize>true</visualize>
+        <update_rate>20</update_rate>
+        <ray>
+            <scan>
+                <horizontal>
+                    <samples>1</samples>
+                    <min_angle>-0.01</min_angle>
+                    <max_angle>0.01</max_angle>
+                </horizontal>
+            </scan>
+            <range>
+                <min>0.02</min>
+                <max>100.0</max>
+                <resolution>0.01</resolution>
+            </range>
+            <noise>
+                <type>gaussian</type>
+                <mean>0.0</mean>
+                <stddev>0.0</stddev>
+            </noise>
+        </ray>
+        <plugin name="gazebo_ros_range" filename="libgazebo_ros_ray_sensor.so">
+            <frame_name>ultrasonic_link</frame_name>
+            <radiation_type>ultrasound</radiation_type>
+            <fov>0.2</fov>
+        </plugin>
+    </sensor>
+  </gazebo>
   <!-- Bring in simulation data for Gazebo. -->
   <xacro:if value="$(arg is_sim)">

Commit message: add non-colliding grass patches and blade controller to control a blade actuator

File: jackal_ws/src/jackal/jackal_description/urdf/jackal.urdf.xacro (robot description, xacro)
@@ -254,4 +254,9 @@
       <state_interface name="position"/>
       <state_interface name="velocity"/>
+    </joint>
+    <joint name="blade_joint">
+        <command_interface name="velocity"/>
+        <state_interface name="position"/>
+        <state_interface name="velocity"/>
     </joint>
   </ros2_control>
@@ -308,4 +313,41 @@
     </sensor>
   </gazebo>
+  <!-- Blade link -->
+  <link name="blade_link">
+    <visual>
+      <origin xyz="0 0 0" rpy="0 0 0"/>
+      <geometry>
+        <box size="0.4 0.05 0.01"/> <!-- long, thin blade -->
+      </geometry>
+      <material name="yellow"/>
+    </visual>
+    <inertial>
+      <mass value="0.1"/>
+      <origin xyz="0 0 0" rpy="0 0 0"/>
+      <inertia ixx="0.0001" ixy="0.0" ixz="0.0" iyy="0.0001" iyz="0.0" izz="0.0001"/>
+    </inertial>
+    <visual>
+        <origin xyz="0 0 0" rpy="0 0 1.5708"/> <!-- 90 degree rotated -->
+        <geometry>
+            <box size="0.4 0.05 0.01"/>
+        </geometry>
+        <material name="yellow"/>
+    </visual>
+  </link>
+  <joint name="blade_joint" type="continuous">
+    <parent link="chassis_link"/>
+    <child link="blade_link"/>
+    <origin xyz="0 0 -0.02" rpy="0 0 0"/> <!-- Adjust height if needed -->
+    <axis xyz="0 0 1"/>
+  </joint>
+  <transmission name="blade_transmission">
+    <type>transmission_interface/SimpleTransmission</type>
+    <joint name="blade_joint">
+      <hardwareInterface>hardware_interface/VelocityJointInterface</hardwareInterface>
+    </joint>
+    <actuator name="blade_motor">
+      <mechanicalReduction>1</mechanicalReduction>
+    </actuator>
+  </transmission>
   <!-- Bring in simulation data for Gazebo. -->
   <xacro:if value="$(arg is_sim)">
