Commit message: working lidar and slam config updates

File: jackal_ws/src/jackal/jackal_description/urdf/accessories/hokuyo_ust10.urdf.xacro (robot description, xacro)
@@ -2,5 +2,5 @@
 <robot xmlns:xacro="http://ros.org/wiki/xacro">
   <xacro:macro name="hokuyo_ust10_mount" params="prefix topic parent_link *origin">
-    <xacro:macro name="hokuyo_ust10" params="frame:=laser topic:=scan sample_size:=720 update_rate:=50
+    <xacro:macro name="hokuyo_ust10" params="frame:=laser topic:=scan sample_size:=720 update_rate:=10
                min_angle:=-2.35619 max_angle:=2.35619 min_range:=0.1 max_range:=30.0 robot_namespace:=/">
       <link name="${frame}">
